File: pindriver.sch (KiCad schematic (older format))
At the start: 0 parts

Commit message: Adds to schematic
Duplicates pin drivers x40, adds connectors.
Parts:
- added P1, P10, P2, P3, P4, P5, P6, P7, P8, P9: CONN_01X20, Connectors_Samtec:SL-120-X-XX_1x20, symbol CONN_01X20
- added P11, P12: CONN_01X03, Connectors_Samtec:SL-103-X-XX_1x03, symbol CONN_01X03
Connections:
- new net EN_GND1: P5.1 (P1)
- new net EN_GND10: P5.10 (P10)
- new net EN_GND11: P5.11 (P11)
- new net EN_GND12: P5.12 (P12)
- new net EN_GND13: P5.13 (P13)
- new net EN_GND14: P5.14 (P14)
- new net EN_GND15: P5.15 (P15)
- new net EN_GND16: P5.16 (P16)
- new net EN_GND17: P5.17 (P17)
- new net EN_GND18: P5.18 (P18)
- new net EN_GND19: P5.19 (P19)
- new net EN_GND2: P5.2 (P2)
- new net EN_GND20: P5.20 (P20)
- new net EN_GND21: P6.1 (P1)
- new net EN_GND22: P6.2 (P2)
- new net EN_GND23: P6.3 (P3)
- new net EN_GND24: P6.4 (P4)
- new net EN_GND25: P6.5 (P5)
- new net EN_GND26: P6.6 (P6)
- new net EN_GND27: P6.7 (P7)
- new net EN_GND28: P6.8 (P8)
- new net EN_GND29: P6.9 (P9)
- new net EN_GND3: P5.3 (P3)
- new net EN_GND30: P6.10 (P10)
- new net EN_GND31: P6.11 (P11)
- new net EN_GND32: P6.12 (P12)
- new net EN_GND33: P6.13 (P13)
- new net EN_GND34: P6.14 (P14)
- new net EN_GND35: P6.15 (P15)
- new net EN_GND36: P6.16 (P16)
- new net EN_GND37: P6.17 (P17)
- new net EN_GND38: P6.18 (P18)
- new net EN_GND39: P6.19 (P19)
- new net EN_GND4: P5.4 (P4)
- new net EN_GND40: P6.20 (P20)
- new net EN_GND5: P5.5 (P5)
- new net EN_GND6: P5.6 (P6)
- new net EN_GND7: P5.7 (P7)
- new net EN_GND8: P5.8 (P8)
- new net EN_GND9: P5.9 (P9)
- new net EN_VDD1: P7.1 (P1)
- new net EN_VDD10: P7.10 (P10)
- new net EN_VDD11: P7.11 (P11)
- new net EN_VDD12: P7.12 (P12)
- new net EN_VDD13: P7.13 (P13)
- new net EN_VDD14: P7.14 (P14)
- new net EN_VDD15: P7.15 (P15)
- new net EN_VDD16: P7.16 (P16)
- new net EN_VDD17: P7.17 (P17)
- new net EN_VDD18: P7.18 (P18)
- new net EN_VDD19: P7.19 (P19)
- new net EN_VDD2: P7.2 (P2)
- new net EN_VDD20: P7.20 (P20)
- new net EN_VDD21: P8.1 (P1)
- new net EN_VDD22: P8.2 (P2)
- new net EN_VDD23: P8.3 (P3)
- new net EN_VDD24: P8.4 (P4)
- new net EN_VDD25: P8.5 (P5)
- new net EN_VDD26: P8.6 (P6)
- new net EN_VDD27: P8.7 (P7)
- new net EN_VDD28: P8.8 (P8)
- new net EN_VDD29: P8.9 (P9)
- new net EN_VDD3: P7.3 (P3)
- new net EN_VDD30: P8.10 (P10)
- new net EN_VDD31: P8.11 (P11)
- new net EN_VDD32: P8.12 (P12)
- new net EN_VDD33: P8.13 (P13)
- new net EN_VDD34: P8.14 (P14)
- new net EN_VDD35: P8.15 (P15)
- new net EN_VDD36: P8.16 (P16)
- new net EN_VDD37: P8.17 (P17)
- new net EN_VDD38: P8.18 (P18)
- new net EN_VDD39: P8.19 (P19)
- new net EN_VDD4: P7.4 (P4)
- new net EN_VDD40: P8.20 (P20)
- new net EN_VDD5: P7.5 (P5)
- new net EN_VDD6: P7.6 (P6)
- new net EN_VDD7: P7.7 (P7)
- new net EN_VDD8: P7.8 (P8)
- new net EN_VDD9: P7.9 (P9)
- new net EN_VPP1: P9.1 (P1)
- new net EN_VPP10: P9.10 (P10)
- new net EN_VPP11: P9.11 (P11)
- new net EN_VPP12: P9.12 (P12)
- new net EN_VPP13: P9.13 (P13)
- new net EN_VPP14: P9.14 (P14)
- new net EN_VPP15: P9.15 (P15)
- new net EN_VPP16: P9.16 (P16)
- new net EN_VPP17: P9.17 (P17)
- new net EN_VPP18: P9.18 (P18)
- new net EN_VPP19: P9.19 (P19)
- new net EN_VPP2: P9.2 (P2)
- new net EN_VPP20: P9.20 (P20)
- new net EN_VPP21: P10.1 (P1)
- new net EN_VPP22: P10.2 (P2)
- new net EN_VPP23: P10.3 (P3)
- new net EN_VPP24: P10.4 (P4)
- new net EN_VPP25: P10.5 (P5)
- new net EN_VPP26: P10.6 (P6)
- new net EN_VPP27: P10.7 (P7)
- new net EN_VPP28: P10.8 (P8)
- new net EN_VPP29: P10.9 (P9)
- new net EN_VPP3: P9.3 (P3)
- new net EN_VPP30: P10.10 (P10)
- new net EN_VPP31: P10.11 (P11)
- new net EN_VPP32: P10.12 (P12)
- new net EN_VPP33: P10.13 (P13)
- new net EN_VPP34: P10.14 (P14)
- new net EN_VPP35: P10.15 (P15)
- new net EN_VPP36: P10.16 (P16)
- new net EN_VPP37: P10.17 (P17)
- new net EN_VPP38: P10.18 (P18)
- new net EN_VPP39: P10.19 (P19)
- new net EN_VPP4: P9.4 (P4)
- new net EN_VPP40: P10.20 (P20)
- new net EN_VPP5: P9.5 (P5)
- new net EN_VPP6: P9.6 (P6)
- new net EN_VPP7: P9.7 (P7)
- new net EN_VPP8: P9.8 (P8)
- new net EN_VPP9: P9.9 (P9)
- new net GNDREF: P11.3 (P3), P12.3 (P3)
- new net PIN1: P1.1 (P1)
- new net PIN10: P1.10 (P10)
- new net PIN11: P1.11 (P11)
- new net PIN12: P1.12 (P12)
- new net PIN13: P1.13 (P13)
- new net PIN14: P1.14 (P14)
- new net PIN15: P1.15 (P15)
- new net PIN16: P1.16 (P16)
- new net PIN17: P1.17 (P17)
- new net PIN18: P1.18 (P18)
- new net PIN19: P1.19 (P19)
- new net PIN2: P1.2 (P2)
- new net PIN20: P1.20 (P20)
- new net PIN21: P2.1 (P1)
- new net PIN22: P2.2 (P2)
- new net PIN23: P2.3 (P3)
- new net PIN24: P2.4 (P4)
- new net PIN25: P2.5 (P5)
- new net PIN26: P2.6 (P6)
- new net PIN27: P2.7 (P7)
- new net PIN28: P2.8 (P8)
- new net PIN29: P2.9 (P9)
- new net PIN3: P1.3 (P3)
- new net PIN30: P2.10 (P10)
- new net PIN31: P2.11 (P11)
- new net PIN32: P2.12 (P12)
- new net PIN33: P2.13 (P13)
- new net PIN34: P2.14 (P14)
- new net PIN35: P2.15 (P15)
- new net PIN36: P2.16 (P16)
- new net PIN37: P2.17 (P17)
- new net PIN38: P2.18 (P18)
- new net PIN39: P2.19 (P19)
- new net PIN4: P1.4 (P4)
- new net PIN40: P2.20 (P20)
- new net PIN5: P1.5 (P5)
- new net PIN6: P1.6 (P6)
- new net PIN7: P1.7 (P7)
- new net PIN8: P1.8 (P8)
- new net PIN9: P1.9 (P9)
- new net SENSE1: P3.1 (P1)
- new net SENSE10: P3.10 (P10)
- new net SENSE11: P3.11 (P11)
- new net SENSE12: P3.12 (P12)
- new net SENSE13: P3.13 (P13)
- new net SENSE14: P3.14 (P14)
- new net SENSE15: P3.15 (P15)
- new net SENSE16: P3.16 (P16)
- new net SENSE17: P3.17 (P17)
- new net SENSE18: P3.18 (P18)
- new net SENSE19: P3.19 (P19)
- new net SENSE2: P3.2 (P2)
- new net SENSE20: P3.20 (P20)
- new net SENSE21: P4.1 (P1)
- new net SENSE22: P4.2 (P2)
- new net SENSE23: P4.3 (P3)
- new net SENSE24: P4.4 (P4)
- new net SENSE25: P4.5 (P5)
- new net SENSE26: P4.6 (P6)
- new net SENSE27: P4.7 (P7)
- new net SENSE28: P4.8 (P8)
- new net SENSE29: P4.9 (P9)
- new net SENSE3: P3.3 (P3)
- new net SENSE30: P4.10 (P10)
- new net SENSE31: P4.11 (P11)
- new net SENSE32: P4.12 (P12)
- new net SENSE33: P4.13 (P13)
- new net SENSE34: P4.14 (P14)
- new net SENSE35: P4.15 (P15)
- new net SENSE36: P4.16 (P16)
- new net SENSE37: P4.17 (P17)
- new net SENSE38: P4.18 (P18)
- new net SENSE39: P4.19 (P19)
- new net SENSE4: P3.4 (P4)
- new net SENSE40: P4.20 (P20)
- new net SENSE5: P3.5 (P5)
- new net SENSE6: P3.6 (P6)
- new net SENSE7: P3.7 (P7)
- new net SENSE8: P3.8 (P8)
- new net SENSE9: P3.9 (P9)
- new net VDD: P11.1 (P1), P12.1 (P1)
- new net VPP: P11.2 (P2), P12.2 (P2)
Other:
- note added: "EN_GND"
- note added: "EN_VDD"
- note added: "EN_VPP"
- note added: "PIN"
- note added: "SENSE"
