File: pindriver.kicad_pcb (KiCad board)
At the start: 2 copper layers, 812 parts, among them P1 CONN_01X20, P10 CONN_01X20, P11 CONN_01X03, P12 CONN_01X03, P2 CONN_01X20, P3 CONN_01X20, P4 CONN_01X20, P5 CONN_01X20, P6 CONN_01X20, P7 CONN_01X20, P8 CONN_01X20, P9 CONN_01X20, Q1 MMBT3904, Q10 BF820, Q100 BF820, Q101 MMBT3904, Q102 MMBT3904, Q103 BF824, Q104 BF824, Q105 BF820, Q106 MMBT3904, Q107 MMBT3904, Q108 BF824, Q109 BF824, Q11 MMBT3904, Q110 BF820, Q111 MMBT3904, Q112 MMBT3904, Q113 BF824, Q114 BF824, Q115 BF820, Q116 MMBT3904, Q117 MMBT3904, Q118 BF824, Q119 BF824, Q12 MMBT3904, Q120 BF820, Q121 MMBT3904, Q122 MMBT3904, Q123 BF824, Q124 BF824, Q125 BF820, Q126 MMBT3904, Q127 MMBT3904, Q128 BF824, Q129 BF824, Q13 BF824, Q130 BF820, Q131 MMBT3904, Q132 MMBT3904, Q133 BF824, Q134 BF824, Q135 BF820, Q136 MMBT3904, Q137 MMBT3904, Q138 BF824, Q139 BF824, Q14 BF824, Q140 BF820, Q141 MMBT3904, Q142 MMBT3904, Q143 BF824, Q144 BF824, Q145 BF820, Q146 MMBT3904, Q147 MMBT3904, Q148 BF824, Q149 BF824, Q15 BF820, Q150 BF820, Q151 MMBT3904, Q152 MMBT3904, Q153 BF824, Q154 BF824, Q155 BF820, Q156 MMBT3904, Q157 MMBT3904, Q158 BF824, Q159 BF824, Q16 MMBT3904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

Commit message: Adds hacked-together PCB parser to duplicate layout, updates simulation with better circuit
Parts:
- moved P10 664.0 mm to (322.6, 111.8), turned to 180 degrees
- moved P8 638.7 mm to (309.9, 114.3), turned to 180 degrees
- moved P6 610.6 mm to (294.6, 114.3), turned to 180 degrees
- moved R212 560.0 mm to (262.9, 133.4), turned to 180 degrees
- moved Q97 559.1 mm to (258.0, 141.0), turned to 180 degrees
- moved Q96 550.7 mm to (258.0, 135.2), turned to 180 degrees
- moved R211 546.9 mm to (262.9, 142.1)
- moved Q98 546.7 mm to (244.5, 136.0), turned to 180 degrees
- moved R217 542.3 mm to (249.6, 141.0), turned to 90 degrees
- moved R210 541.4 mm to (262.9, 136.2)
- moved D39 535.8 mm to (234.7, 136.2), turned to 90 degrees
- moved R213 534.9 mm to (262.9, 139.3), turned to 180 degrees
- moved R215 533.6 mm to (252.8, 142.3)
- moved Q100 532.7 mm to (238.8, 135.8), turned to 180 degrees
- moved R216 532.5 mm to (249.6, 135.8), turned to 90 degrees
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Routing:
- net /PIN2: track 0.00 -> 111.9 mm
- net /PIN1: track 0.00 -> 78.5 mm
- net /SENSE1: track 0.00 -> 61.9 mm
- net /PIN3: track 0.00 -> 40.5 mm
- net Net-(C71-Pad1): track 0.00 -> 8.61 mm
- net Net-(C72-Pad1): track 0.00 -> 8.56 mm
- net Net-(Q180-Pad2): track 0.00 -> 7.27 mm
- net Net-(C71-Pad2): track 0.00 -> 6.86 mm
- net Net-(C72-Pad2): track 0.00 -> 6.45 mm
- net Net-(Q177-Pad1): track 0.00 -> 6.15 mm
- net Net-(Q176-Pad1): track 0.00 -> 6.15 mm
- net Net-(D72-Pad2): track 0.00 -> 5.42 mm
- net VDD: track 0.00 -> 3.74 mm
- net VPP: track 0.00 -> 3.70 mm
- net Net-(D72-Pad1): track 0.00 -> 3.11 mm
